Commit message: Modify name to ur3e in my_moveit_config due to mismatch with real robot. use_sim_time set to false

File: my_moveit_config/config/ur3e.ros2_control.xacro (robot description, xacro)
@@ -1,5 +1,5 @@
 <?xml version="1.0"?>
 <robot xmlns:xacro="http://www.ros.org/wiki/xacro">
-    <xacro:macro name="name_ros2_control" params="name initial_positions_file">
+    <xacro:macro name="ur3e_ros2_control" params="name initial_positions_file">
         <xacro:property name="initial_positions" value="${load_yaml(initial_positions_file)['initial_positions']}"/>
         <ros2_control name="${name}" type="system">

File: my_moveit_config/config/ur3e.urdf.xacro (robot description, xacro)
@@ -1,11 +1,11 @@
 <?xml version="1.0"?>
-<robot xmlns:xacro="http://www.ros.org/wiki/xacro" name="name">
+<robot xmlns:xacro="http://www.ros.org/wiki/xacro" name="ur3e">
     <xacro:arg name="my_initial_positions_file"
            default="$(find my_moveit_config)/config/initial_positions.yaml" />
-    <!-- Import name urdf file -->
+    <!-- Import URDF file -->
     <xacro:include filename="$(find ur_description)/urdf/ur.urdf.xacro" />
     <!-- Import control_xacro -->
-    <xacro:include filename="name.ros2_control.xacro" />
-    <xacro:name_ros2_control
+    <xacro:include filename="ur3e.ros2_control.xacro" />
+    <xacro:ur3e_ros2_control
     name="FakeSystem"
     initial_positions_file="$(arg my_initial_positions_file)" />
