Commit message: Set OMPL+PILZ architecture

File: my_moveit_config/config/name.ros2_control.xacro (robot description, xacro)
@@ -2,5 +2,5 @@
 <robot xmlns:xacro="http://www.ros.org/wiki/xacro">
     <xacro:macro name="name_ros2_control" params="name initial_positions_file">
-        <xacro:property name="initial_positions" value="${xacro.load_yaml(initial_positions_file)['initial_positions']}"/>
+        <xacro:property name="initial_positions" value="${load_yaml(initial_positions_file)['initial_positions']}"/>
         <ros2_control name="${name}" type="system">
             <hardware>

Commit message: Fixed model name clash between name and ur3e

File: my_moveit_config/config/name.ros2_control.xacro (robot description, xacro)
@@ -1,6 +1,7 @@
 <?xml version="1.0"?>
 <robot xmlns:xacro="http://www.ros.org/wiki/xacro">
-    <xacro:macro name="ur3e_ros2_control" params="name initial_positions_file">
-        <xacro:property name="initial_positions" value="${load_yaml(initial_positions_file)['initial_positions']}"/>
+    <xacro:macro name="name_ros2_control" params="name initial_positions_file">
+        <xacro:property name="raw_initial_positions" value="${xacro.load_yaml(initial_positions_file)}"/>
+        <xacro:property name="initial_positions" value="${raw_initial_positions['initial_positions'] if 'initial_positions' in raw_initial_positions else raw_initial_positions}"/>
         <ros2_control name="${name}" type="system">
             <hardware>

Commit message: Adapted -sim working commit into -main real robot lab

File: my_moveit_config/config/name.ros2_control.xacro (robot description, xacro)
@@ -2,5 +2,6 @@
 <robot xmlns:xacro="http://www.ros.org/wiki/xacro">
     <xacro:macro name="name_ros2_control" params="name initial_positions_file">
-        <xacro:property name="initial_positions" value="${load_yaml(initial_positions_file)['initial_positions']}"/>
+        <xacro:property name="raw_initial_positions" value="${xacro.load_yaml(initial_positions_file)}"/>
+        <xacro:property name="initial_positions" value="${raw_initial_positions['initial_positions'] if 'initial_positions' in raw_initial_positions else raw_initial_positions}"/>
         <ros2_control name="${name}" type="system">
             <hardware>

File: my_moveit_config/config/name.urdf.xacro (robot description, xacro)
@@ -1,12 +1,9 @@
 <?xml version="1.0"?>
 <robot xmlns:xacro="http://www.ros.org/wiki/xacro" name="name">
-    <xacro:arg name="my_initial_positions_file"
-           default="$(find my_moveit_config)/config/initial_positions.yaml" />
+    <xacro:arg name="initial_positions_file" default="$(find my_moveit_config)/config/initial_positions.yaml" />
     <!-- Import name urdf file -->
     <xacro:include filename="$(find ur_description)/urdf/ur.urdf.xacro" />
     <!-- Import control_xacro -->
     <xacro:include filename="name.ros2_control.xacro" />
-    <xacro:name_ros2_control
-    name="FakeSystem"
-    initial_positions_file="$(arg my_initial_positions_file)" />
+    <xacro:name_ros2_control name="FakeSystem" initial_positions_file="$(arg initial_positions_file)"/>
 </robot>
